Commit message: add RPP control

File: diff_tracked/diff_tracked_base/urdf/imu_driver.xacro (robot description, xacro)
@@ -10,5 +10,5 @@
         <topicName>/imu</topicName>
         <bodyName>imu_link</bodyName>
-        <updateRateHZ>100.0</updateRateHZ>
+        <updateRateHZ>300.0</updateRateHZ>
         <gaussianNoise>0.0</gaussianNoise>
         <xyzOffset>0 0 0</xyzOffset>

File: diff_tracked/diff_tracked_base/urdf/laser_driver.xacro (robot description, xacro)
@@ -10,5 +10,5 @@
         <scan>
           <horizontal>
-            <samples>1800</samples>
+            <samples>900</samples>
             <resolution>1</resolution>
             <min_angle>-${3.141592653589793}</min_angle>

File: diff_tracked/diff_tracked_gazebo/urdf/bunker.xacro (robot description, xacro)
@@ -40,9 +40,12 @@
     <collision>
       <origin
-        xyz="0.53 -0.392 -0.358"
-        rpy="1.57 0 3.14" />
-      <geometry>
-        <mesh
-          filename="package://diff_tracked_base/meshes/BUNKER.STL" scale="0.001 0.001 0.001" />
+        xyz="0 0 -0.12"
+        rpy="0 0 0" />
+      <geometry>
+        <!-- The original BUNKER mesh includes the tracks down to z=-0.358 m.
+             Using it as the chassis collision keeps the driven wheels above
+             the ground.  A raised chassis collision lets the road wheels
+             carry the vehicle while preserving the mesh as the visual. -->
+        <box size="0.90 0.60 0.25" />
       </geometry>
     </collision>
@@ -90,5 +93,5 @@
   <joint
     name="wheel1_joint"
-    type="revolute">
+    type="continuous">
     <origin
       xyz="0.44403 0.3495 -0.12853"
@@ -101,8 +104,6 @@
       xyz="0 0 1" />
     <limit
-      lower="-180"
-      upper="180"
-      effort="0"
-      velocity="0" />
+      effort="30"
+      velocity="20" />
   </joint>
   <link
@@ -148,5 +149,5 @@
   <joint
     name="wheel1.1_jont"
-    type="revolute">
+    type="continuous">
     <origin
       xyz="0.37551 0.3495 -0.22305"
@@ -159,8 +160,6 @@
       xyz="0 0 1" />
     <limit
-      lower="-180"
-      upper="180"
-      effort="0"
-      velocity="0" />
+      effort="30"
+      velocity="20" />
   </joint>
   <link
@@ -206,5 +205,5 @@
   <joint
     name="wheel1.2_joint"
-    type="revolute">
+    type="continuous">
     <origin
       xyz="0.29039 0.3495 -0.28104"
@@ -217,8 +216,6 @@
       xyz="0 0 1" />
     <limit
-      lower="-180"
-      upper="180"
-      effort="0"
-      velocity="0" />
+      effort="30"
+      velocity="20" />
   </joint>
   <link
@@ -264,5 +261,5 @@
   <joint
     name="wheel1.3_joint"
-    type="revolute">
+    type="continuous">
     <origin
       xyz="0.29603 0.3495 -0.087"
@@ -275,8 +272,6 @@
       xyz="0 0 -1" />
     <limit
-      lower="-180"
-      upper="180"
-      effort="0"
-      velocity="0" />
+      effort="30"
+      velocity="20" />
   </joint>
   <link
@@ -322,5 +317,5 @@
   <joint
     name="wheel2_joint"
-    type="revolute">
+    type="continuous">
     <origin
       xyz="0.44403 -0.3495 -0.12853"
@@ -333,8 +328,6 @@
       xyz="0 0 -1" />
     <limit
-      lower="-180"
-      upper="180"
-      effort="0"
-      velocity="0" />
+      effort="30"
+      velocity="20" />
   </joint>
   <link
@@ -380,5 +373,5 @@
   <joint
     name="wheel2.1_joint"
-    type="revolute">
+    type="continuous">
     <origin
       xyz="0.37551 -0.3495 -0.22305"
@@ -391,8 +384,6 @@
       xyz="0 0 -1" />
     <limit
-      lower="-180"
-      upper="180"
-      effort="0"
-      velocity="0" />
+      effort="30"
+      velocity="20" />
   </joint>
   <link
@@ -438,5 +429,5 @@
   <joint
     name="wheel2.2_joint"
-    type="revolute">
+    type="continuous">
     <origin
       xyz="0.29039 -0.3495 -0.28104"
@@ -447,10 +438,8 @@
       link="wheel2.2_Link" />
     <axis
-      xyz="0 0 -1" />
-    <limit
-      lower="-180"
-      upper="180"
-      effort="0"
-      velocity="0" />
+      xyz="0 0 1" />
+    <limit
+      effort="30"
+      velocity="20" />
   </joint>
   <link
@@ -496,5 +485,5 @@
   <joint
     name="wheel2.3_joint"
-    type="revolute">
+    type="continuous">
     <origin
       xyz="0.29603 -0.3495 -0.087"
@@ -507,8 +496,6 @@
       xyz="0 0 1" />
     <limit
-      lower="-180"
-      upper="180"
-      effort="0"
-      velocity="0" />
+      effort="30"
+      velocity="20" />
   </joint>
   <link
@@ -554,5 +541,5 @@
   <joint
     name="wheel3_joint"
-    type="revolute">
+    type="continuous">
     <origin
       xyz="-0.38871 0.295 -0.19381"
@@ -565,8 +552,6 @@
       xyz="0 0 -1" />
     <limit
-      lower="-180"
-      upper="180"
-      effort="0"
-      velocity="0" />
+      effort="30"
+      velocity="20" />
   </joint>
   <link
@@ -612,5 +597,5 @@
   <joint
     name="wheel3.1_joint"
-    type="revolute">
+    type="continuous">
     <origin
       xyz="-0.23111 0.3495 -0.27671"
@@ -623,8 +608,6 @@
       xyz="0 0 1" />
     <limit
-      lower="-180"
-      upper="180"
-      effort="0"
-      velocity="0" />
+      effort="30"
+      velocity="20" />
   </joint>
   <link
@@ -670,5 +653,5 @@
   <joint
     name="wheel3.2_joint"
-    type="revolute">
+    type="continuous">
     <origin
       xyz="0.043885 0.3495 -0.27671"
@@ -681,8 +664,6 @@
       xyz="0 0 1" />
     <limit
-      lower="-180"
-      upper="180"
-      effort="0"
-      velocity="0" />
+      effort="30"
+      velocity="20" />
   </joint>
   <link
@@ -728,5 +709,5 @@
   <joint
     name="wheel3.3_joint"
-    type="revolute">
+    type="continuous">
     <origin
       xyz="-0.28597 0.3495 -0.087"
@@ -739,8 +720,6 @@
       xyz="0 0 -1" />
     <limit
-      lower="-180"
-      upper="180"
-      effort="0"
-      velocity="0" />
+      effort="30"
+      velocity="20" />
   </joint>
   <link
@@ -786,5 +765,5 @@
   <joint
     name="wheel4_joint"
-    type="revolute">
+    type="continuous">
     <origin
       xyz="-0.38871 -0.295 -0.19381"
@@ -797,8 +776,6 @@
       xyz="0 0 1" />
     <limit
-      lower="-180"
-      upper="180"
-      effort="0"
-      velocity="0" />
+      effort="30"
+      velocity="20" />
   </joint>
   <link
@@ -844,5 +821,5 @@
   <joint
     name="wheel4.1_joint"
-    type="revolute">
+    type="continuous">
     <origin
       xyz="-0.23111 -0.3495 -0.27671"
@@ -855,8 +832,6 @@
       xyz="0 0 -1" />
     <limit
-      lower="-180"
-      upper="180"
-      effort="0"
-      velocity="0" />
+      effort="30"
+      velocity="20" />
   </joint>
   <link
@@ -902,5 +877,5 @@
   <joint
     name="wheel4.2_joint"
-    type="revolute">
+    type="continuous">
     <origin
       xyz="0.043885 -0.3495 -0.27671"
@@ -913,8 +888,6 @@
       xyz="0 0 -1" />
     <limit
-      lower="-180"
-      upper="180"
-      effort="0"
-      velocity="0" />
+      effort="30"
+      velocity="20" />
   </joint>
   <link
@@ -960,5 +933,5 @@
   <joint
     name="wheel4.3_joint"
-    type="revolute">
+    type="continuous">
     <origin
       xyz="-0.28597 -0.3495 -0.087"
@@ -971,8 +944,6 @@
       xyz="0 0 1" />
     <limit
-      lower="-180"
-      upper="180"
-      effort="0"
-      velocity="0" />
+      effort="30"
+      velocity="20" />
   </joint>
   <!-- /////////////////////////////////   gazebo color   ////////////////////////////////////// -->
@@ -989,5 +960,5 @@
     </plugin>
   </gazebo> -->
-  <gazebo>
+  <!-- <gazebo>
     <plugin name="object_controller" filename="libgazebo_ros_planar_move.so">
       <commandTopic>cmd_vel</commandTopic>
@@ -1001,11 +972,66 @@
       <robotBaseFrame>base_link</robotBaseFrame>
     </plugin>
+  </gazebo> -->
+  <gazebo>
+    <plugin name="gazebo_ros_diff_drive" filename="libgazebo_ros_diff_drive.so">
+      <legacyMode>false</legacyMode>
+      <updateRate>100.0</updateRate>
+      <leftJoint>wheel1.2_joint</leftJoint>
+      <rightJoint>wheel2.2_joint</rightJoint>
+      <wheelSeparation>0.699</wheelSeparation>
+      <wheelDiameter>0.102</wheelDiameter>
+      <wheelTorque>30.0</wheelTorque>
+      <wheelAcceleration>1.8</wheelAcceleration>
+      <commandTopic>cmd_vel</commandTopic>
+      <odometryTopic>odom</odometryTopic>
+      <odometryFrame>odom</odometryFrame>
+      <robotBaseFrame>base_link</robotBaseFrame>
+      <publishOdom>true</publishOdom>
+      <publishOdomTF>false</publishOdomTF>
+      <publishWheelTF>false</publishWheelTF>
+      <publishWheelJointState>false</publishWheelJointState>
+    </plugin>
+  </gazebo>
+  <gazebo reference="wheel1.2_Link">
+    <mu1>1.0</mu1>
+    <mu2>1.0</mu2>
+    <kp>100000.0</kp>
+    <kd>1.0</kd>
+  </gazebo>
+  <gazebo reference="wheel2.2_Link">
+    <mu1>1.0</mu1>
+    <mu2>1.0</mu2>
+    <kp>100000.0</kp>
+    <kd>1.0</kd>
   </gazebo>
   <gazebo>
+  <plugin name="joint_state_publisher"
+          filename="libgazebo_ros_joint_state_publisher.so">
+    <updateRate>50</updateRate>
+    <jointName>
+      wheel1_joint,
+      wheel1.1_jont,
+      wheel1.2_joint,
+      wheel1.3_joint,
+      wheel2_joint,
+      wheel2.1_joint,
+      wheel2.2_joint,
+      wheel2.3_joint,
+      wheel3_joint,
+      wheel3.1_joint,
+      wheel3.2_joint,
+      wheel3.3_joint,
+      wheel4_joint,
+      wheel4.1_joint,
+      wheel4.2_joint,
+      wheel4.3_joint
+    </jointName>
+  </plugin>
+</gazebo>
+  <!-- <gazebo>
     <plugin name="gazebo_ros_control" filename="libgazebo_ros_control.so">
-      <!-- <robotNamespace>/</robotNamespace> -->
       <robotSimType>gazebo_ros_control/DefaultRobotHWSim</robotSimType>
       <legacyModeNS>true</legacyModeNS>
     </plugin>
-  </gazebo>
+  </gazebo> -->
 </robot>
