Commit message: add robot-localization

File: diff_tracked/diff_tracked_base/urdf/bunker_laser_3d.xacro (robot description, xacro)
@@ -1,7 +1,13 @@
 <robot name="bunker_laser_3d"
   xmlns:xacro="http://wiki.ros.org/xacro">
+  <xacro:arg name="use_3d_lidar" default="false"/>
+  <xacro:if value="$(arg use_3d_lidar)">
+    <xacro:include filename="laser_3d_driver.xacro"/>
+  </xacro:if>
+  <xacro:unless value="$(arg use_3d_lidar)">
+    <xacro:include filename="laser_2d_driver.xacro"/>
+  </xacro:unless>
   <xacro:include filename="bunker.xacro" />
   <xacro:include filename="laser.xacro" />
-  <xacro:include filename="laser_3d_driver.xacro" />
   <xacro:include filename="imu.xacro" />
   <xacro:include filename="imu_driver.xacro" />

File: diff_tracked/diff_tracked_base/urdf/imu_driver.xacro (robot description, xacro)
@@ -8,8 +8,10 @@
       <pose>0 0 0 0 0 0</pose>
       <plugin name="tracked_imu_plugin" filename="libgazebo_ros_imu_sensor.so">
-        <topicName>/imu</topicName>
+        <!-- The virtual encoder node republishes this as /imu with
+             independently configurable covariance. -->
+        <topicName>/imu_raw</topicName>
         <bodyName>imu</bodyName>
         <updateRateHZ>100.0</updateRateHZ>
-        <gaussianNoise>0.0</gaussianNoise>
+        <gaussianNoise>0.001</gaussianNoise>
         <xyzOffset>0 0 0</xyzOffset>
         <rpyOffset>0 0 0</rpyOffset>

File: diff_tracked/diff_tracked_base/urdf/laser.xacro (robot description, xacro)
@@ -7,5 +7,5 @@
   <xacro:property name="laser_x" value="0.0"/>
   <xacro:property name="laser_y" value="0.0"/>
-  <xacro:property name="laser_z" value="${laser_length / 2}"/>
+  <xacro:property name="laser_z" value="${laser_length / 2 + 0.04}"/>
   <link name="laser">
     <inertial>

File: diff_tracked/diff_tracked_base/urdf/move.xacro (robot description, xacro)
@@ -5,5 +5,5 @@
       <commandTopic>/cmd_vel</commandTopic>
       <odometryTopic>/gz_odom</odometryTopic>
-      <odometryFrame>world</odometryFrame>
+      <odometryFrame>odom</odometryFrame>
       <robotBaseFrame>base_link</robotBaseFrame>
       <odometryRate>100.0</odometryRate>
